Commit message: Shrunk the robot (length: 0.8). Fixed positions of wheels, etc... & moved bottom cameras to centre

File: src/my_robot_description/urdf/cameraBL.xacro (robot description, xacro)
@@ -22,5 +22,5 @@
         <parent link="base_link" />
         <child link="camera_linkBL" />
-        <origin xyz="${((base_length + camera_length) / 2.0) - 0.1} 0.1 ${base_height / 2.0 - 0.3}" rpy="0 ${pi/2} 0" />
+        <origin xyz="0 0.1 ${base_height / 2.0 - 0.305}" rpy="0 ${pi/2} 0" />
     </joint>
     <link name="camera_link_opticalBL" />

File: src/my_robot_description/urdf/cameraBM.xacro (robot description, xacro)
@@ -22,5 +22,5 @@
         <parent link="base_link" />
         <child link="camera_linkBM" />
-        <origin xyz="${((base_length + camera_length) / 2.0) - 0.1} 0 ${base_height / 2.0 - 0.3}" rpy="0 ${pi/2} 0" />
+        <origin xyz="0 0 ${base_height / 2.0 - 0.305}" rpy="0 ${pi/2} 0" />
     </joint>
     <link name="camera_link_opticalBM" />

File: src/my_robot_description/urdf/cameraBR.xacro (robot description, xacro)
@@ -22,5 +22,5 @@
         <parent link="base_link" />
         <child link="camera_linkBR" />
-        <origin xyz="${((base_length + camera_length) / 2.0) - 0.1} -0.1 ${base_height / 2.0 - 0.3}" rpy="0 ${pi/2} 0" />
+        <origin xyz="0 -0.1 ${base_height / 2.0 - 0.305}" rpy="0 ${pi/2} 0" />
     </joint>
     <link name="camera_link_opticalBR" />

File: src/my_robot_description/urdf/mobile_base.xacro (robot description, xacro)
@@ -2,5 +2,5 @@
 <robot xmlns:xacro="http://www.ros.org/wiki/xacro">
     <!-- Updated properties to match your robot model -->
-    <xacro:property name="base_length" value="1.0"/>
+    <xacro:property name="base_length" value="0.8"/>
     <xacro:property name="base_width"  value="0.6"/>
     <xacro:property name="base_height" value="0.3"/>
@@ -43,5 +43,5 @@
         <parent link="base_link"/>
         <child link="front_box_link"/>
-        <origin xyz="0.23 0 0.29" rpy="0 0 0"/>
+        <origin xyz="0.18 0 0.20" rpy="0 0 0"/>
     </joint>
     <link name="front_box_link">
@@ -49,5 +49,5 @@
             <origin xyz="0 0 0" rpy="0 0 0"/>
             <geometry>
-                <box size="0.4 0.4 0.3"/>
+                <box size="0.3 0.3 0.25"/>
             </geometry>
             <material name="accent_orange">
@@ -68,5 +68,5 @@
         <parent link="base_link"/>
         <child link="basket_back_link"/>
-        <origin xyz="-0.45 0 0.2" rpy="0 0 0"/>
+        <origin xyz="-0.35 0 0.2" rpy="0 0 0"/>
     </joint>
     <link name="basket_back_link">
@@ -84,5 +84,5 @@
         <parent link="base_link"/>
         <child link="basket_left_link"/>
-        <origin xyz="-0.3 0.2 0.2" rpy="0 0 0"/>
+        <origin xyz="-0.2 0.2 0.2" rpy="0 0 0"/>
     </joint>
     <link name="basket_left_link">
@@ -100,5 +100,5 @@
         <parent link="base_link"/>
         <child link="basket_right_link"/>
-        <origin xyz="-0.3 -0.2 0.2" rpy="0 0 0"/>
+        <origin xyz="-0.2 -0.2 0.2" rpy="0 0 0"/>
     </joint>
     <link name="basket_right_link">
@@ -116,5 +116,5 @@
         <parent link="base_link"/>
         <child link="basket_front_link"/>
-        <origin xyz="-0.15 0 0.2" rpy="0 0 0"/>
+        <origin xyz="-0.05 0 0.2" rpy="0 0 0"/>
     </joint>
     <link name="basket_front_link">
@@ -133,5 +133,5 @@
         <parent link="base_link"/>
         <child link="light1_link"/>
-        <origin xyz="0.5 -0.15 0" rpy="0 -1.5708 0"/>
+        <origin xyz="${(base_length + 0.01) / 2.0} -0.15 0" rpy="0 -1.5708 0"/>
     </joint>
     <link name="light1_link">
@@ -139,5 +139,5 @@
             <origin xyz="0 0 0" rpy="0 0 0"/>
             <geometry>
-                <cylinder length="0.1" radius="0.05"/>
+                <cylinder length="0.01" radius="0.05"/>
             </geometry>
             <material name="headlight_warm">
@@ -149,5 +149,5 @@
         <parent link="base_link"/>
         <child link="light2_link"/>
-        <origin xyz="0.5 0.15 0" rpy="0 -1.5708 0"/>
+        <origin xyz="${(base_length + 0.01) / 2.0} 0.15 0" rpy="0 -1.5708 0"/>
     </joint>
     <link name="light2_link">
@@ -155,5 +155,5 @@
             <origin xyz="0 0 0" rpy="0 0 0"/>
             <geometry>
-                <cylinder length="0.1" radius="0.05"/>
+                <cylinder length="0.01" radius="0.05"/>
             </geometry>
             <material name="headlight_warm">
@@ -191,5 +191,5 @@
         <parent link="base_link"/>
         <child link="rear_left_wheel_link"/>
-        <origin xyz="-0.3 0.32 -0.1" rpy="0 0 0"/>
+        <origin xyz="${(-(base_length + 0.01) / 2.0) + 0.2} 0.32 -0.1" rpy="0 0 0"/>
         <axis xyz="0 1 0"/>
     </joint>
@@ -197,5 +197,5 @@
         <parent link="base_link"/>
         <child link="rear_right_wheel_link"/>
-        <origin xyz="-0.3 -0.32 -0.1" rpy="0 0 0"/>
+        <origin xyz="${(-(base_length + 0.01) / 2.0) + 0.2} -0.32 -0.1" rpy="0 0 0"/>
         <axis xyz="0 1 0"/>
     </joint>
@@ -206,5 +206,5 @@
         <parent link="base_link"/>
         <child link="front_right_wheel_link"/>
-        <origin xyz="0.3 -0.32 -0.1" rpy="0 0 0"/>
+        <origin xyz="${((base_length + 0.01) / 2.0) - 0.2} -0.32 -0.1" rpy="0 0 0"/>
         <axis xyz="0 1 0"/>
     </joint>
@@ -230,5 +230,5 @@
         <parent link="base_link"/>
         <child link="front_left_wheel_link"/>
-        <origin xyz="0.3 0.32 -0.1" rpy="0 0 0"/>
+        <origin xyz="${((base_length + 0.01) / 2.0) - 0.2} 0.32 -0.1" rpy="0 0 0"/>
         <axis xyz="0 1 0"/>
     </joint>

Commit message: current version (side cameras are IN the side wheels)

File: src/my_robot_description/urdf/cameraBL.xacro (robot description, xacro)
@@ -22,5 +22,5 @@
         <parent link="base_link" />
         <child link="camera_linkBL" />
-        <origin xyz="0 0.2 ${base_height / 2.0 - 0.305}" rpy="0 ${pi/2} 0" />
+        <origin xyz="0 0.2 ${base_height / 2.0 - 0.31}" rpy="0 ${pi/2} 0" />
     </joint>
     <link name="camera_link_opticalBL" />

File: src/my_robot_description/urdf/cameraBM.xacro (robot description, xacro)
@@ -22,5 +22,5 @@
         <parent link="base_link" />
         <child link="camera_linkBM" />
-        <origin xyz="0 0 ${base_height / 2.0 - 0.305}" rpy="0 ${pi/2} 0" />
+        <origin xyz="0 0 ${base_height / 2.0 - 0.31}" rpy="0 ${pi/2} 0" />
     </joint>
     <link name="camera_link_opticalBM" />

File: src/my_robot_description/urdf/cameraBR.xacro (robot description, xacro)
@@ -22,5 +22,5 @@
         <parent link="base_link" />
         <child link="camera_linkBR" />
-        <origin xyz="0 -0.2 ${base_height / 2.0 - 0.305}" rpy="0 ${pi/2} 0" />
+        <origin xyz="0 -0.2 ${base_height / 2.0 - 0.31}" rpy="0 ${pi/2} 0" />
     </joint>
     <link name="camera_link_opticalBR" />
