Commit message: Moved the wheels down and in

File: src/my_robot_description/urdf/mobile_base.xacro (robot description, xacro)
@@ -191,5 +191,5 @@
         <parent link="base_link"/>
         <child link="rear_left_wheel_link"/>
-        <origin xyz="${(-(base_length + 0.01) / 2.0) + 0.2} ${base_width/2.0} -0.15" rpy="0 0 0"/>
+        <origin xyz="${(-(base_length + 0.01) / 2.0) + 0.15} ${(base_width/2.0) - 0.03} -0.2" rpy="0 0 0"/>
         <axis xyz="0 1 0"/>
     </joint>
@@ -197,5 +197,5 @@
         <parent link="base_link"/>
         <child link="rear_right_wheel_link"/>
-        <origin xyz="${(-(base_length + 0.01) / 2.0) + 0.2} -${base_width/2.0} -0.15" rpy="0 0 0"/>
+        <origin xyz="${(-(base_length + 0.01) / 2.0) + 0.15} -${(base_width/2.0) - 0.03} -0.2" rpy="0 0 0"/>
         <axis xyz="0 1 0"/>
     </joint>
@@ -206,5 +206,5 @@
         <parent link="base_link"/>
         <child link="front_right_wheel_link"/>
-        <origin xyz="${((base_length + 0.01) / 2.0) - 0.2} -${base_width/2.0} -0.15" rpy="0 0 0"/>
+        <origin xyz="${((base_length + 0.01) / 2.0) - 0.15} -${(base_width/2.0) - 0.03} -0.2" rpy="0 0 0"/>
         <axis xyz="0 1 0"/>
     </joint>
@@ -230,5 +230,5 @@
         <parent link="base_link"/>
         <child link="front_left_wheel_link"/>
-        <origin xyz="${((base_length + 0.01) / 2.0) - 0.2} ${base_width/2.0} -0.15" rpy="0 0 0"/>
+        <origin xyz="${((base_length + 0.01) / 2.0) - 0.15} ${(base_width/2.0) - 0.03} -0.2" rpy="0 0 0"/>
         <axis xyz="0 1 0"/>
     </joint>

Commit message: changed urdf
- made front wheels frictionless
- raised the whole robot 0.15m so it doesn't get stuck in the floor.

File: src/my_robot_description/urdf/mobile_base.xacro (robot description, xacro)
@@ -15,5 +15,5 @@
         <parent link="base_footprint"/>
         <child link="base_link"/>
-        <origin xyz="0 0 0.15"/>
+        <origin xyz="0 0 0.2"/>
     </joint>
     <!-- =============== -->
@@ -191,5 +191,5 @@
         <parent link="base_link"/>
         <child link="rear_left_wheel_link"/>
-        <origin xyz="${(-(base_length + 0.01) / 2.0) + 0.15} ${(base_width/2.0) - 0.03} -0.2" rpy="0 0 0"/>
+        <origin xyz="${(-(base_length + 0.01) / 2.0) + 0.15} ${(base_width/2.0) - 0.03} -0.05" rpy="0 0 0"/>
         <axis xyz="0 1 0"/>
     </joint>
@@ -197,5 +197,5 @@
         <parent link="base_link"/>
         <child link="rear_right_wheel_link"/>
-        <origin xyz="${(-(base_length + 0.01) / 2.0) + 0.15} -${(base_width/2.0) - 0.03} -0.2" rpy="0 0 0"/>
+        <origin xyz="${(-(base_length + 0.01) / 2.0) + 0.15} -${(base_width/2.0) - 0.03} -0.05" rpy="0 0 0"/>
         <axis xyz="0 1 0"/>
     </joint>
@@ -206,5 +206,5 @@
         <parent link="base_link"/>
         <child link="front_right_wheel_link"/>
-        <origin xyz="${((base_length + 0.01) / 2.0) - 0.15} -${(base_width/2.0) - 0.03} -0.2" rpy="0 0 0"/>
+        <origin xyz="${((base_length + 0.01) / 2.0) - 0.15} -${(base_width/2.0) - 0.03} -0.05" rpy="0 0 0"/>
         <axis xyz="0 1 0"/>
     </joint>
@@ -230,5 +230,5 @@
         <parent link="base_link"/>
         <child link="front_left_wheel_link"/>
-        <origin xyz="${((base_length + 0.01) / 2.0) - 0.15} ${(base_width/2.0) - 0.03} -0.2" rpy="0 0 0"/>
+        <origin xyz="${((base_length + 0.01) / 2.0) - 0.15} ${(base_width/2.0) - 0.03} -0.05" rpy="0 0 0"/>
         <axis xyz="0 1 0"/>
     </joint>

File: src/my_robot_description/urdf/mobile_base_gazebo.xacro (robot description, xacro)
@@ -10,11 +10,12 @@
         <mu2 value="0.2" />
     </gazebo>
+    <!--slippery front wheels-->
     <gazebo reference="front_left_wheel_link">
-        <mu1 value="1.0" />
-        <mu2 value="0.2" />
+        <mu1 value="0.1" />
+        <mu2 value="0.1" />
     </gazebo>
     <gazebo reference="front_right_wheel_link">
-        <mu1 value="1.0" />
-        <mu2 value="0.2" />
+        <mu1 value="0.1" />
+        <mu2 value="0.1" />
     </gazebo>
     <!-- Differential Drive Plugin -->
@@ -25,5 +26,5 @@
             <left_joint>rear_left_wheel_joint</left_joint>
             <right_joint>rear_right_wheel_joint</right_joint>
-            <wheel_separation>0.64</wheel_separation>
+            <wheel_separation>0.44</wheel_separation>
             <wheel_radius>0.15</wheel_radius>
             <frame_id>odom</frame_id>

Commit message: some changes
- fixed the gemini code
- the cameras are being obscured though, gonna fix that now

File: src/my_robot_description/urdf/mobile_base.xacro (robot description, xacro)
@@ -188,18 +188,4 @@
     <xacro:rear_wheel_link prefix="rear_left"/>
     <xacro:rear_wheel_link prefix="rear_right"/>
-    <!--
-    <joint name="rear_left_wheel_joint" type="continuous">
-        <parent link="base_link"/>
-        <child link="rear_left_wheel_link"/>
-        <origin xyz="${(-(base_length + 0.01) / 2.0) + 0.15} ${(base_width/2.0) - 0.03} -0.05" rpy="0 0 0"/>
-        <axis xyz="0 1 0"/>
-    </joint>
-    <joint name="rear_right_wheel_joint" type="continuous">
-        <parent link="base_link"/>
-        <child link="rear_right_wheel_link"/>
-        <origin xyz="${(-(base_length + 0.01) / 2.0) + 0.15} -${(base_width/2.0) - 0.03} -0.05" rpy="0 0 0"/>
-        <axis xyz="0 1 0"/>
-    </joint>
-    -->
     <joint name="rear_left_wheel_joint" type="continuous">
         <parent link="base_link"/>
@@ -215,56 +201,6 @@
     </joint>
     <!-- ============================ -->
-    <!-- Front Wheels (Fixed)        -->
-    <!-- ============================ -->
-    <!--
-    <link name="front_right_wheel_link">
-        <visual>
-            <origin rpy="${pi/2} 0 0" xyz="0 0 0"/>
-            <geometry>
-                <cylinder length="${wheel_length}" radius="${wheel_radius}"/>
-            </geometry>
-            <material name="rubber_black">
-                <color rgba="0.06 0.06 0.06 1.0"/>
-            </material>
-        </visual>
-        <collision>
-            <geometry>
-                <sphere radius="${wheel_radius}"/>
-            </geometry>
-        </collision>
-        <xacro:cylinder_inertia m="1.0" r="${wheel_radius}" l="${wheel_length}"
-                                o_xyz="0 0 0" o_rpy="${pi/2.0} 0 0"/>
-    </link>
-    <link name="front_left_wheel_link">
-        <visual>
-            <origin rpy="${pi/2} 0 0" xyz="0 0 0"/>
-            <geometry>
-                <cylinder length="${wheel_length}" radius="${wheel_radius}"/>
-            </geometry>
-            <material name="rubber_black">
-                <color rgba="0.06 0.06 0.06 1.0"/>
-            </material>
-        </visual>
-        <collision>
-            <geometry>
-                <sphere radius="${wheel_radius}"/>
-            </geometry>
-        </collision>
-        <xacro:cylinder_inertia m="1.0" r="${wheel_radius}" l="${wheel_length}"
-                                o_xyz="0 0 0" o_rpy="${pi/2.0} 0 0"/>
-    </link>
-    <joint name="front_left_wheel_joint" type="continuous">
-        <parent link="base_link"/>
-        <child link="front_left_wheel_link"/>
-        <origin xyz="${((base_length + 0.01) / 2.0) - 0.15} ${(base_width/2.0) - 0.03} -0.05" rpy="0 0 0"/>
-        <axis xyz="0 1 0"/>
-    </joint>
-    <joint name="front_right_wheel_joint" type="continuous">
-        <parent link="base_link"/>
-        <child link="front_right_wheel_link"/>
-        <origin xyz="${((base_length + 0.01) / 2.0) - 0.15} -${(base_width/2.0) - 0.03} -0.05" rpy="0 0 0"/>
-        <axis xyz="0 1 0"/>
-    </joint>
-    -->
+    <!-- Caster Wheels                -->
+    <!-- ============================ -->
     <joint name="front_caster_joint" type="fixed">
         <parent link="base_link"/>
@@ -278,5 +214,8 @@
         </visual>
         <collision>
-            <geometry><sphere radius="${wheel_radius}"/></collision>
+            <geometry>
+            <sphere radius="${wheel_radius}"/>
+            </geometry>
+        </collision>
         <xacro:sphere_inertia m="0.5" r="${wheel_radius}" o_xyz="0 0 0" o_rpy="0 0 0"/>
     </link>
@@ -292,5 +231,6 @@
         </visual>
         <collision>
-            <geometry><sphere radius="${wheel_radius}"/></collision>
+            <geometry><sphere radius="${wheel_radius}"/></geometry>
+        </collision>
         <xacro:sphere_inertia m="0.5" r="${wheel_radius}" o_xyz="0 0 0" o_rpy="0 0 0"/>
     </link>

File: src/my_robot_description/urdf/mobile_base_gazebo.xacro (robot description, xacro)
@@ -11,14 +11,4 @@
     </gazebo>
     <!--slippery front wheels-->
-    <!--
-    <gazebo reference="front_left_wheel_link">
-        <mu1 value="0.000" />
-        <mu2 value="0.000" />
-    </gazebo>
-    <gazebo reference="front_right_wheel_link">
-        <mu1 value="0.000" />
-        <mu2 value="0.000" />
-    </gazebo>
-    -->
     <gazebo reference="front_caster_link">
         <mu1 value="0.0"/><mu2 value="0.0"/>
@@ -34,5 +24,5 @@
             <left_joint>rear_left_wheel_joint</left_joint>
             <right_joint>rear_right_wheel_joint</right_joint>
-            <wheel_separation>0.72</wheel_separation>
+            <wheel_separation>0.44</wheel_separation>
             <wheel_radius>0.15</wheel_radius>
             <max_wheel_torque>100</max_wheel_torque>
@@ -49,6 +39,6 @@
             <joint_name>rear_left_wheel_joint</joint_name>
             <joint_name>rear_right_wheel_joint</joint_name>
-            <joint_name>front_left_wheel_joint</joint_name>
-            <joint_name>front_right_wheel_joint</joint_name>
+            <joint_name>rear_caster_joint</joint_name>
+            <joint_name>front_caster_joint</joint_name>
         </plugin>
     </gazebo>

Commit message: Adjust wheel joint origins and radius calculations
Updated joint origins and sphere radius for caster wheels.

File: src/my_robot_description/urdf/mobile_base.xacro (robot description, xacro)
@@ -191,5 +191,5 @@
         <parent link="base_link"/>
         <child link="rear_left_wheel_link"/>
-        <origin xyz="0 ${(base_width/2.0) - 0.03} -0.05" rpy="0 0 0"/>
+        <origin xyz="0 ${(base_width/2.0) + 0.03} -0.125" rpy="0 0 0"/>
         <axis xyz="0 1 0"/>
     </joint>
@@ -197,5 +197,5 @@
         <parent link="base_link"/>
         <child link="rear_right_wheel_link"/>
-        <origin xyz="0 ${-(base_width/2.0) + 0.03} -0.05" rpy="0 0 0"/>
+        <origin xyz="0 ${-(base_width/2.0) - 0.03} -0.125" rpy="0 0 0"/>
         <axis xyz="0 1 0"/>
     </joint>
@@ -206,32 +206,32 @@
         <parent link="base_link"/>
         <child link="front_caster_link"/>
-        <origin xyz="0.3 0 -0.05" rpy="0 0 0"/>
+        <origin xyz="0.3 0 -0.175" rpy="0 0 0"/>
     </joint>
     <link name="front_caster_link">
         <visual>
-            <geometry><sphere radius="${wheel_radius}"/></geometry>
+            <geometry><sphere radius="${wheel_radius/1.5}"/></geometry>
             <material name="rubber_black"><color rgba="0.1 0.1 0.1 1"/></material>
         </visual>
         <collision>
             <geometry>
-            <sphere radius="${wheel_radius}"/>
-            </geometry>
-        </collision>
-        <xacro:sphere_inertia m="0.5" r="${wheel_radius}" o_xyz="0 0 0" o_rpy="0 0 0"/>
+            <sphere radius="${wheel_radius/1.5}"/>
+            </geometry>
+        </collision>
+        <xacro:sphere_inertia m="0.5" r="${wheel_radius/1.5}" o_xyz="0 0 0" o_rpy="0 0 0"/>
     </link>
     <joint name="rear_caster_joint" type="fixed">
         <parent link="base_link"/>
         <child link="rear_caster_link"/>
-        <origin xyz="-0.3 0 -0.05" rpy="0 0 0"/>
+        <origin xyz="-0.3 0 -0.175" rpy="0 0 0"/>
     </joint>
     <link name="rear_caster_link">
         <visual>
-            <geometry><sphere radius="${wheel_radius}"/></geometry>
+            <geometry><sphere radius="${wheel_radius/1.5}"/></geometry>
             <material name="rubber_black"><color rgba="0.1 0.1 0.1 1"/></material>
         </visual>
         <collision>
-            <geometry><sphere radius="${wheel_radius}"/></geometry>
-        </collision>
-        <xacro:sphere_inertia m="0.5" r="${wheel_radius}" o_xyz="0 0 0" o_rpy="0 0 0"/>
+            <geometry><sphere radius="${wheel_radius/1.5}"/></geometry>
+        </collision>
+        <xacro:sphere_inertia m="0.5" r="${wheel_radius/1.5}" o_xyz="0 0 0" o_rpy="0 0 0"/>
     </link>
 </robot>
