Commit message: restart line_following

File: src/my_robot_description/urdf/camera.xacro (robot description, xacro)
@@ -22,5 +22,5 @@
         <parent link="base_link" />
         <child link="camera_link" />
-        <origin xyz="${(base_length + camera_length) / 2.0} 0 ${base_height / 2.0 - 0.1}" rpy="0 0 0" />
+        <origin xyz="${(base_length + camera_length) / 2.0} 0 ${base_height / 2.0 - 0.1}" rpy="0 0.4 0" />
     </joint>
     <link name="camera_link_optical" />
